Commit message: Start example with ee wrench

File: test/test_data/robot_with_visuals.urdf (robot description, URDF)
Before this commit: robot robot_arm, 8 links, 7 joints
Links:
- link link1: geometry visual cylinder length=0.14 radius=0.05
- link link2: geometry visual cylinder length=0.1 radius=0.05; visual cylinder length=0.28 radius=0.05
- link link4: geometry visual cylinder length=0.34 radius=0.05
- link link6: geometry visual cylinder length=0.05 radius=0.05
