Commit message: Scale mesh

File: test/test_data/simple_mechanism.urdf (robot description, URDF)
Before this commit: robot simple_mechanism, 2 links, 1 joints
Links:
- link lower_cone: geometry visual mesh filename=cone.stl scale=1 1 0.5
- link upper_cone: geometry visual mesh filename=cone.stl scale=1 1 0.5

Commit message: Fix visualizer example
No motion was previously visible because of the choice of the joint
axis.

File: test/test_data/simple_mechanism.urdf (robot description, URDF)
Before this commit: robot simple_mechanism, 2 links, 1 joints
Joints:
- joint joint: axis 1 0 0 -> 0 1 0
